Commit message: modeled the robot

File: description/core.xacro (robot description, xacro)
@@ -39,4 +39,9 @@
         </xacro:inertial_box>
     </link>
+    <gazebo reference="chassis">
+        <material>
+            Gazebo/White
+        </material>
+    </gazebo>
     <joint name="left_wheel_joint" type="continuous">
         <parent link="base_link"/>
@@ -61,4 +66,9 @@
         </xacro:inertial_cylinder>
     </link>
+    <gazebo reference="left_wheel">
+        <material>
+            Gazebo/Blue
+        </material>
+    </gazebo>
     <joint name="right_wheel_joint" type="continuous">
         <parent link="base_link"/>
@@ -83,4 +93,9 @@
         </xacro:inertial_cylinder>
     </link>
+    <gazebo reference="right_wheel">
+        <material>
+            Gazebo/Orange
+        </material>
+    </gazebo>
     <joint name="caster_wheel_joint" type="fixed">
         <parent link="chassis"/>
@@ -104,3 +119,10 @@
         </xacro:inertial_sphere>
     </link>
+    <gazebo reference="caster_wheel">
+        <material>
+            Gazebo/White
+        </material>
+        <mu1 value="0.001"></mu1>
+        <mu2 value="0.001"></mu2>
+    </gazebo>
 </robot>

File: description/robot.urdf.xacro (robot description, xacro)
@@ -2,3 +2,4 @@
 <robot xmlns:xacro="http://www.ros.org/wiki/xacro"  name="robot">
     <xacro:include filename="core.xacro" />
+    <xacro:include filename="gazebo_control.xacro"/>
 </robot>
